Commit message: added caster wheels

File: urdf/barista_robot_model.urdf (robot description, URDF)
Before this commit: robot barista_robot, 7 links, 6 joints
Links:
- added link back_pitch_link; visual sphere radius=0.0352
- added link back_roll_link; visual cylinder length=0.010 radius=0.0352
- added link back_yaw_link; visual cylinder length=0.005 radius=0.0352
- added link front_pitch_link; visual sphere radius=0.0352
- added link front_roll_link; visual cylinder length=0.010 radius=0.0352
- added link front_yaw_link; visual cylinder length=0.005 radius=0.0352
- added link left_wheel; visual cylinder length=0.0206 radius=0.0352
- added link right_wheel; visual cylinder length=0.0206 radius=0.0352
Joints:
- added joint back_pitch_joint: type continuous, parent back_roll_link, child back_pitch_link, origin xyz=0 0 0 rpy=0 0 0, axis 0 1 0, limit effort=1000.0 velocity=100.0
- added joint back_roll_joint: type continuous, parent back_yaw_link, child back_roll_link, origin xyz=0 0 0 rpy=0 0 0, axis 1 0 0, limit effort=1000.0 velocity=100.0
- added joint back_yaw_joint: type continuous, parent chassis, child back_yaw_link, origin xyz=0.0 -0.12 -0.070 rpy=0 0 0, axis 0 0 1, limit effort=1000.0 velocity=100.0
- added joint front_pitch_joint: type continuous, parent front_roll_link, child front_pitch_link, origin xyz=0 0 0 rpy=0 0 0, axis 0 1 0, limit effort=1000.0 velocity=100.0
- added joint front_roll_joint: type continuous, parent front_yaw_link, child front_roll_link, origin xyz=0 0 0 rpy=0 0 0, axis 1 0 0, limit effort=1000.0 velocity=100.0
- added joint front_yaw_joint: type continuous, parent chassis, child front_yaw_link, origin xyz=0.0 0.12 -0.070 rpy=0 0 0, axis 0 0 1, limit effort=1000.0 velocity=100.0
- added joint joint_left_wheel: type continuous, parent chassis, child left_wheel, origin xyz=0.14 0.0 -0.070 rpy=0 0 0, axis 0 1 0, limit effort=10000 velocity=1000
- added joint joint_right_wheel: type continuous, parent chassis, child right_wheel, origin xyz=-0.14 0.0 -0.070 rpy=0 0 0, axis 0 1 0, limit effort=10000 velocity=1000

Commit message: corrected wheel and caster wheels orientation. facing jitter issue when controlled through joint state publisher

File: urdf/barista_robot_model.urdf (robot description, URDF)
Before this commit: robot barista_robot, 15 links, 14 joints
Links:
- removed link back_pitch_link
- removed link front_pitch_link
- added link front_text; visual box size=0.01 0.02 0.01
- added link laser_link, mass 0.3; collision cylinder length=0.04 radius=0.025; visual cylinder length=0.04 radius=0.025
- link back_roll_link: mass None -> 0.1; geometry collision sphere radius=0.0352; visual sphere radius=0.0352
- link back_yaw_link: mass None -> 0.1; geometry collision cylinder length=0.005 radius=0.01; visual cylinder length=0.005 radius=0.01
- link base_link: geometry 
- link chassis: mass None -> 5.0
- link cup_holder_tray: mass None -> 1.0
- link front_roll_link: mass None -> 0.2; geometry collision sphere radius=0.0352; visual sphere radius=0.0352
- link front_yaw_link: mass None -> 0.1; geometry collision cylinder length=0.005 radius=0.01; visual cylinder length=0.005 radius=0.01
- link left_wheel: mass None -> 0.5
- link right_wheel: mass None -> 0.5
- link standoff_back_left: mass None -> 0.1
- link standoff_back_right: mass None -> 0.1
- link standoff_front_left: mass None -> 0.1
- link standoff_front_right: mass None -> 0.1
Joints:
- removed joint back_pitch_joint
- removed joint front_pitch_joint
- added joint joint_front_text: type fixed, parent chassis, child front_text, origin xyz=0.18 0.0 0.0 rpy=0.0 0.0 0.0
- added joint joint_laser: type fixed, parent chassis, child laser_link, origin xyz=0.15 0.0 0.095 rpy=0.0 0.0 0.0
- joint back_yaw_joint: origin xyz=0.0 -0.12 -0.070 rpy=0 0 0 -> xyz=-0.12 0.0 -0.070 rpy=0 0 0
- joint base_link_joint: origin xyz=0.0 0.0 0.0 rpy=0.0 0.0 0.0 -> xyz=0.0 0.0 0.0775 rpy=0.0 0.0 0.0
- joint front_yaw_joint: origin xyz=0.0 0.12 -0.070 rpy=0 0 0 -> xyz=0.12 0.0 -0.070 rpy=0 0 0
- joint joint_left_wheel: origin xyz=0.14 0.0 -0.070 rpy=0 0 0 -> xyz=0.0 0.14 -0.070 rpy=0 0 0
- joint joint_right_wheel: origin xyz=-0.14 0.0 -0.070 rpy=0 0 0 -> xyz=0.0 -0.14 -0.070 rpy=0 0 0
- joint joint_standoff_back_left: origin xyz=0 0.0 0.1875 rpy=0 0 0 -> xyz=-0.065 0.12 0.1875 rpy=0 0 0
- joint joint_standoff_back_right: origin xyz=0 0.0 0.1875 rpy=0 0 0 -> xyz=-0.065 -0.12 0.1875 rpy=0 0 0
- joint joint_standoff_front_left: origin xyz=0 0.0 0.1875 rpy=0 0 0 -> xyz=0.065 0.12 0.1875 rpy=0 0 0
- joint joint_standoff_front_right: origin xyz=0 0.0 0.1875 rpy=0 0 0 -> xyz=0.065 -0.12 0.1875 rpy=0 0 0

Commit message: laser sick time551(mesh) added. fixed some joint origins for wheels and casterwheels

File: urdf/barista_robot_model.urdf (robot description, URDF)
Before this commit: robot barista_robot, 15 links, 14 joints
Links:
- removed link front_text
- added link front_indicator; visual box size=0.01 0.02 0.01
- link laser_link: geometry collision mesh filename=package://barista_robot_description/meshes/sick_tim551.dae scale=0.6 0.6 0.6; visual mesh filename=package://barista_robot_description/meshes/sick_tim551.dae scale=0.6 0.6 0.6
Joints:
- removed joint joint_front_text
- added joint joint_front_indicator: type fixed, parent chassis, child front_indicator, origin xyz=0.18 0.0 0.0 rpy=0.0 0.0 0.0
- joint joint_laser: origin xyz=0.15 0.0 0.095 rpy=0.0 0.0 0.0 -> xyz=0.15 0.0 0.077 rpy=0.0 0.0 0.0

Commit message: Changes in caster wheel type (continous to fixed). Added gazebo material

File: urdf/barista_robot_model.urdf (robot description, URDF)
Before this commit: robot barista_robot, 15 links, 14 joints
Links:
- removed link front_indicator
- added link back_pitch_link, mass 0.1; collision cylinder length=0.010 radius=0.0352; visual sphere radius=0.0352
- added link front_pitch_link, mass 0.1; collision cylinder length=0.010 radius=0.0352; visual sphere radius=0.0352
- link back_roll_link: geometry collision cylinder length=0.010 radius=0.0352; visual cylinder length=0.010 radius=0.0352
- link back_yaw_link: geometry collision cylinder length=0.010 radius=0.0352; visual cylinder length=0.010 radius=0.0352
- link chassis: mass 5.0 -> 0.8; geometry collision cylinder length=0.155 radius=0.178; visual cylinder length=0.155 radius=0.178
- link front_roll_link: mass 0.2 -> 0.1; geometry collision cylinder length=0.010 radius=0.0352; visual cylinder length=0.010 radius=0.0352
- link front_yaw_link: mass 0.1 -> None; geometry visual cylinder length=0.010 radius=0.0352
- link left_wheel: mass 0.5 -> 0.07; geometry collision cylinder length=0.010 radius=0.0352; visual cylinder length=0.0206 radius=0.0352
- link right_wheel: mass 0.5 -> 0.07; geometry collision cylinder length=0.010 radius=0.0352; visual cylinder length=0.0206 radius=0.0352
Joints:
- removed joint joint_front_indicator
- added joint back_pitch_joint: type fixed, parent back_roll_link, child back_pitch_link, origin xyz=0 0 0 rpy=0 1.5707 1.5707, axis 0 1 0, limit effort=1000.0 velocity=100.0
- added joint front_pitch_joint: type fixed, parent front_roll_link, child front_pitch_link, origin xyz=0 0 0 rpy=0 1.5707 1.5707, axis 0 1 0, limit effort=1000.0 velocity=100.0
- joint back_roll_joint: origin xyz=0 0 0 rpy=0 0 0 -> xyz=0 0 0 rpy=0 1.5707 1.5707; type continuous -> fixed
- joint back_yaw_joint: axis 0 0 1 -> 0 1 0; origin xyz=-0.12 0.0 -0.070 rpy=0 0 0 -> xyz=-0.12 0.0 -0.070 rpy=0 1.5707 1.5707; type continuous -> fixed
- joint front_roll_joint: origin xyz=0 0 0 rpy=0 0 0 -> xyz=0 0 0 rpy=0 1.5707 1.5707; type continuous -> fixed
- joint front_yaw_joint: axis 0 0 1 -> 0 1 0; origin xyz=0.12 0.0 -0.070 rpy=0 0 0 -> xyz=0.12 0.0 -0.070 rpy=0 1.5707 1.5707; type continuous -> fixed
- joint joint_left_wheel: origin xyz=0.0 0.14 -0.070 rpy=0 0 0 -> xyz=0.0 0.14 -0.070 rpy=1.5707 0 0
- joint joint_right_wheel: origin xyz=0.0 -0.14 -0.070 rpy=0 0 0 -> xyz=0.0 -0.14 -0.070 rpy=1.5707 0 0

Commit message: Laser plugin and frame corrections

File: urdf/barista_robot_model.urdf (robot description, URDF)
Before this commit: robot barista_robot, 16 links, 15 joints
Links:
- added link laser_optical_frame
- link laser_link: geometry collision mesh filename=package://barista_robot_description/meshes/sick_tim551.dae; visual mesh filename=package://barista_robot_description/meshes/sick_tim551.dae
Joints:
- added joint laser_optical_joint: type fixed, parent laser_link, child laser_optical_frame, origin xyz=0.0 0.0 0.06 rpy=0.0 0.0 0.0
- joint joint_laser: origin xyz=0.15 0.0 0.077 rpy=0.0 0.0 0.0 -> xyz=0.12 0.0 0.077 rpy=0.0 0.0 0.0

Commit message: task2 - Introducing Xacro macros to existing barista urdf file

File: urdf/barista_robot_model.urdf (robot description, URDF)
Before this commit: robot barista_robot, 17 links, 16 joints
Links:
- link left_wheel: geometry collision cylinder length=0.0206 radius=0.0352; visual cylinder length=0.0206 radius=0.0352
- link right_wheel: geometry collision cylinder length=0.0206 radius=0.0352; visual cylinder length=0.0206 radius=0.0352
- link standoff_back_left: geometry collision cylinder length=0.010 radius=0.220; visual cylinder length=0.220 radius=0.010
- link standoff_back_right: geometry collision cylinder length=0.010 radius=0.220; visual cylinder length=0.220 radius=0.010
- link standoff_front_left: geometry collision cylinder length=0.010 radius=0.220; visual cylinder length=0.220 radius=0.010
- link standoff_front_right: geometry collision cylinder length=0.010 radius=0.220; visual cylinder length=0.220 radius=0.010
