Commit message: changes related to caster wheel to accept physics property xacro file

File: xacro/caster_wheel.xacro (robot description, xacro)
@@ -1,6 +1,8 @@
 <?xml version="1.0"?>
 <robot xmlns:xacro="http://www.ros.org/wiki/xacro">
-  <!-- Caster wheel macro -->
-  <xacro:macro name="caster_wheel" params="prefix x_pos robot_name">
+    <!-- Load physics parameters -->
+    <xacro:include filename="$(find barista_robot_description)/xacro/physics_properties.xacro"/>
+    <!-- Caster wheel macro -->
+    <xacro:macro name="caster_wheel" params="prefix x_pos robot_name">
     <!-- Properties -->
     <xacro:property name="wheel_radius" value="0.0352"/>
@@ -23,6 +25,10 @@
         </collision>
         <inertial>
-            <mass value="${wheel_mass}"/>
-            <inertia ixx="0.0000031184" ixy="0" ixz="0" iyy="0.0000031184" iyz="0" izz="0.000006195"/>
+            <!-- <mass value="${wheel_mass}"/>
+            <inertia ixx="0.0000031184" ixy="0" ixz="0" iyy="0.0000031184" iyz="0" izz="0.000006195"/> -->
+            <mass value="${physics_config['caster_mass']}"/>
+            <inertia ixx="${physics_config['caster_yr_ixx']}" ixy="0" ixz="0"
+                     iyy="${physics_config['caster_yr_iyy']}" iyz="0"
+                     izz="${physics_config['caster_yr_izz']}"/>
         </inertial>
     </link>
@@ -34,6 +40,7 @@
         <axis xyz="0 0 1 " />
         <limit effort="1000.0" velocity="100.0" />
-        <!-- <dynamics damping="2.0" friction="0.5"/> -->
-        <dynamics damping="3.0" friction="0.7"/>
+        <!-- <dynamics damping="3.0" friction="0.7"/> -->
+        <dynamics damping="${physics_config['wheel_damping']}"
+                        friction="${physics_config['wheel_friction']}"/>
     </joint>
     <!-- Roll link -->
@@ -51,11 +58,15 @@
         </collision>
         <inertial>
-            <mass value="${wheel_mass}"/>
-            <inertia ixx="0.0000031184" ixy="0" ixz="0" iyy="0.0000031184" iyz="0" izz="0.000006195"/>
+            <!-- <mass value="${wheel_mass}"/>
+            <inertia ixx="0.0000031184" ixy="0" ixz="0" iyy="0.0000031184" iyz="0" izz="0.000006195"/> -->
+            <mass value="${physics_config['caster_mass']}"/>
+            <inertia ixx="${physics_config['caster_yr_ixx']}" ixy="0" ixz="0"
+                     iyy="${physics_config['caster_yr_iyy']}" iyz="0"
+                     izz="${physics_config['caster_yr_izz']}"/>
         </inertial>
     </link>
     <joint name="${prefix}_roll_joint" type="${joint_type}">
         <!-- <origin rpy="0 1.5707 1.5707" xyz="0 0 0" /> -->
-        <origin rpy="0 0 0" xyz="0 0 0" />
+        <origin rpy="0 1.5707 1.5707" xyz="0 0 0" />
         <parent link="${prefix}_yaw_link" />
         <child link="${prefix}_roll_link" />
@@ -63,6 +74,7 @@
         <axis xyz="0 1 0" />
         <limit effort="1000.0" velocity="100.0" />
-        <!-- <dynamics damping="0.5" friction="0.1"/> -->
-        <dynamics damping="1.0" friction="0.5"/>
+        <!-- <dynamics damping="1.0" friction="0.5"/> -->
+        <dynamics damping="${physics_config['wheel_damping']}"
+                        friction="${physics_config['wheel_friction']}"/>
     </joint>
     <!-- Pitch link -->
@@ -80,13 +92,16 @@
         </collision>
         <inertial>
-            <mass value="${wheel_mass}"/>
+            <!-- <mass value="${wheel_mass}"/>
             <inertia ixx="0.00000826" ixy="0" ixz="0"
                      iyy="00.00000826" iyz="0"
-                     izz="0.00000826"/>
+                     izz="0.00000826"/> -->
+            <mass value="${physics_config['caster_mass']}"/>
+            <inertia ixx="${physics_config['caster_p_ixx']}" ixy="0" ixz="0"
+                     iyy="${physics_config['caster_p_iyy']}" iyz="0"
+                     izz="${physics_config['caster_p_izz']}"/>
         </inertial>
     </link>
     <joint name="${prefix}_pitch_joint" type="${joint_type}">
-        <!-- <origin rpy="0 1.5707 1.5707" xyz="0 0 0" /> -->
-        <origin rpy="0 0 0" xyz="0 0 0" />
+        <origin rpy="0 1.5707 1.5707" xyz="0 0 0" />
         <parent link="${prefix}_roll_link" />
         <child link="${prefix}_pitch_link" />
@@ -95,5 +110,7 @@
         <!-- <axis xyz="1 0 0" /> -->
         <limit effort="1000.0" velocity="100.0" />
-        <dynamics damping="0.01" friction="0.01"/>
+        <!-- <dynamics damping="0.01" friction="0.01"/> -->
+        <dynamics damping="${physics_config['wheel_damping']}"
+                        friction="${physics_config['wheel_friction']}"/>
     </joint>
     <!-- Gazebo materials -->

File: xacro/drive_wheel.xacro (robot description, xacro)
@@ -62,6 +62,6 @@
         <limit effort="10000" velocity="1000"/>
         <!-- <joint_properties damping="3.0" friction="0.4"/> -->
-    <joint_properties damping="${physics_config['wheel_damping']}"
-                     friction="${physics_config['wheel_friction']}"/>
+        <joint_properties damping="${physics_config['wheel_damping']}"
+                        friction="${physics_config['wheel_friction']}"/>
     </joint>
   </xacro:macro>
