Commit message: wheel separation, laserScan ray and caster wheels through xacro fixed for Task 2

File: xacro/barista_robot_model.urdf.xacro (robot description, xacro)
@@ -78,5 +78,6 @@
     <!-- Caster Wheels -->
     <xacro:include filename="$(find barista_robot_description)/xacro/caster_wheel.xacro"/>
-    <xacro:caster_wheel/>
+    <xacro:caster_wheel prefix="front" x_pos="0.12"/>
+    <xacro:caster_wheel prefix="back" x_pos="-0.12"/>
     <!-- Cup Holder Tray -->
     <xacro:include filename="$(find barista_robot_description)/xacro/cup_holder_tray.xacro"/>

File: xacro/caster_wheel.xacro (robot description, xacro)
@@ -1,10 +1,12 @@
 <?xml version="1.0"?>
 <robot xmlns:xacro="http://www.ros.org/wiki/xacro">
-  <xacro:macro name="caster_wheel">
-    <!-- Xacro properties for wheel dimensions -->
+  <!-- Caster wheel macro -->
+  <xacro:macro name="caster_wheel" params="prefix x_pos">
+    <!-- Properties -->
     <xacro:property name="wheel_radius" value="0.0352"/>
     <xacro:property name="cylinder_length" value="0.010"/>
-    <!-- Front Caster Wheel -->
-    <link name="front_yaw_link">
+    <xacro:property name="wheel_mass" value="0.1"/>
+    <!-- Yaw link -->
+    <link name="${prefix}_yaw_link">
         <visual>
             <geometry>
@@ -13,10 +15,4 @@
             <material name="green_dark"/>
         </visual>
-        <inertial>
-            <mass value="0.1"/>
-            <inertia ixx="3.1809333333333334e-05" ixy="0" ixz="0"
-                     iyy="3.1809333333333334e-05" iyz="0"
-                     izz="6.1952e-05"/>
-            </inertial>
         <collision>
             <geometry>
@@ -24,14 +20,21 @@
             </geometry>
         </collision>
+        <inertial>
+            <mass value="${wheel_mass}"/>
+            <inertia ixx="3.1809333333333334e-05" ixy="0" ixz="0"
+                     iyy="3.1809333333333334e-05" iyz="0"
+                     izz="6.1952e-05"/>
+        </inertial>
     </link>
-    <joint name="front_yaw_joint" type="fixed">
-        <origin rpy="0 1.5707 1.5707" xyz="0.12 0.0 -0.070" />
+    <joint name="${prefix}_yaw_joint" type="fixed">
+        <origin rpy="0 1.5707 1.5707" xyz="${x_pos} 0.0 -0.070" />
         <parent link="chassis" />
-        <child link="front_yaw_link" />
+        <child link="${prefix}_yaw_link" />
         <axis xyz="0 1 0" />
         <limit effort="1000.0" velocity="100.0" />
         <dynamics damping="0.5" friction="0.5"/>
     </joint>
-    <link name="front_roll_link">
+    <!-- Roll link -->
+    <link name="${prefix}_roll_link">
         <visual>
             <geometry>
@@ -40,10 +43,4 @@
             <material name="green_dark"/>
         </visual>
-        <inertial>
-            <mass value="0.1"/>
-            <inertia ixx="3.1809333333333334e-05" ixy="0" ixz="0"
-                     iyy="3.1809333333333334e-05" iyz="0"
-                     izz="6.1952e-05"/>
-            </inertial>
         <collision>
             <geometry>
@@ -51,26 +48,27 @@
             </geometry>
         </collision>
+        <inertial>
+            <mass value="${wheel_mass}"/>
+            <inertia ixx="3.1809333333333334e-05" ixy="0" ixz="0"
+                     iyy="3.1809333333333334e-05" iyz="0"
+                     izz="6.1952e-05"/>
+        </inertial>
     </link>
-    <joint name="front_roll_joint" type="fixed">
+    <joint name="${prefix}_roll_joint" type="fixed">
         <origin rpy="0 1.5707 1.5707" xyz="0 0 0" />
-        <parent link="front_yaw_link" />
-        <child link="front_roll_link" />
+        <parent link="${prefix}_yaw_link" />
+        <child link="${prefix}_roll_link" />
         <axis xyz="1 0 0" />
         <limit effort="1000.0" velocity="100.0" />
         <dynamics damping="0.5" friction="0.5"/>
     </joint>
-    <link name="front_pitch_link">
+    <!-- Pitch link -->
+    <link name="${prefix}_pitch_link">
         <visual>
             <geometry>
                 <sphere radius="${wheel_radius}"/>
             </geometry>
-        <material name="green_dark"/>
+            <material name="green_dark"/>
         </visual>
-        <inertial>
-            <mass value="0.1"/>
-            <inertia ixx="4.95616e-05" ixy="0" ixz="0"
-                     iyy="4.95616e-05" iyz="0"
-                     izz="4.95616e-05"/>
-            </inertial>
         <collision>
             <geometry>
@@ -78,98 +76,35 @@
             </geometry>
         </collision>
+        <inertial>
+            <origin xyz="0 0 0" rpy="0 0 0"/>
+            <mass value="${wheel_mass}"/>
+            <inertia ixx="4.95616e-05" ixy="0" ixz="0"
+                     iyy="4.95616e-05" iyz="0"
+                     izz="4.95616e-05"/>
+        </inertial>
     </link>
-    <joint name="front_pitch_joint" type="fixed">
+    <joint name="${prefix}_pitch_joint" type="fixed">
         <origin rpy="0 1.5707 1.5707" xyz="0 0 0" />
-        <parent link="front_roll_link" />
-        <child link="front_pitch_link" />
+        <parent link="${prefix}_roll_link" />
+        <child link="${prefix}_pitch_link" />
         <axis xyz="0 1 0" />
         <limit effort="1000.0" velocity="100.0" />
         <dynamics damping="0.5" friction="0.5"/>
     </joint>
-    <!-- Back Caster Wheel -->
-    <link name="back_yaw_link">
-        <visual>
-            <geometry>
-                <cylinder length="${cylinder_length}" radius="${wheel_radius}"/>
-            </geometry>
-            <material name="green_dark"/>
-        </visual>
-        <inertial>
-            <mass value="0.1"/>
-            <inertia ixx="3.1809333333333334e-05" ixy="0" ixz="0"
-                     iyy="3.1809333333333334e-05" iyz="0"
-                     izz="6.1952e-05"/>
-            </inertial>
-        <collision>
-            <geometry>
-                <cylinder length="${cylinder_length}" radius="${wheel_radius}"/>
-            </geometry>
-        </collision>
-    </link>
-    <joint name="back_yaw_joint" type="fixed">
-        <origin rpy="0 1.5707 1.5707" xyz="-0.12 0.0 -0.070" />
-        <parent link="chassis" />
-        <child link="back_yaw_link" />
-        <axis xyz="0 1 0" />
-        <limit effort="1000.0" velocity="100.0" />
-        <dynamics damping="0.5" friction="0.5"/>
-    </joint>
-    <link name="back_roll_link">
-        <visual>
-            <geometry>
-                <cylinder length="${cylinder_length}" radius="${wheel_radius}"/>
-            </geometry>
-            <material name="green_dark"/>
-        </visual>
-        <inertial>
-            <mass value="0.1"/>
-            <inertia ixx="3.1809333333333334e-05" ixy="0" ixz="0"
-                     iyy="3.1809333333333334e-05" iyz="0"
-                     izz="6.1952e-05"/>
-            </inertial>
-        <collision>
-            <geometry>
-                <cylinder length="${cylinder_length}" radius="${wheel_radius}"/>
-            </geometry>
-        </collision>
-    </link>
-    <joint name="back_roll_joint" type="fixed">
-        <origin rpy="0 1.5707 1.5707" xyz="0 0 0" />
-        <parent link="back_yaw_link" />
-        <child link="back_roll_link" />
-        <axis xyz="1 0 0" />
-        <limit effort="1000.0" velocity="100.0" />
-        <dynamics damping="0.5" friction="0.5"/>
-    </joint>
-    <link name="back_pitch_link">
-        <visual>
-            <geometry>
-                <sphere radius="${wheel_radius}"/>
-            </geometry>
-        <material name="green_dark"/>
-        </visual>
-        <inertial>
-            <mass value="0.1"/>
-            <inertia ixx="4.95616e-05" ixy="0" ixz="0"
-                     iyy="4.95616e-05" iyz="0"
-                     izz="4.95616e-05"/>
-            </inertial>
-        <collision>
-            <geometry>
-                <sphere radius="${wheel_radius}"/>
-            </geometry>
-        </collision>
-    </link>
-    <joint name="back_pitch_joint" type="fixed">
-        <origin rpy="0 1.5707 1.5707" xyz="0 0 0" />
-        <parent link="back_roll_link" />
-        <child link="back_pitch_link" />
-        <axis xyz="0 1 0" />
-        <limit effort="1000.0" velocity="100.0" />
-        <dynamics damping="0.5" friction="0.5"/>
-    </joint>
-    <gazebo reference="front_yaw_link">
+    <!-- Gazebo materials -->
+    <gazebo reference="${prefix}_yaw_link">
+        <material>Gazebo/Grey</material>
+    </gazebo>
+    <gazebo reference="${prefix}_roll_link">
+        <material>Gazebo/Grey</material>
+    </gazebo>
+    <gazebo reference="${prefix}_pitch_link">
         <material>Gazebo/Grey</material>
     </gazebo>
   </xacro:macro>
+  <!-- Need to check this way of implementation too -->
+  <!-- <xacro:macro name="caster_wheel">
+    <xacro:caster_wheel prefix="front" x_pos="0.12"/>
+    <xacro:caster_wheel prefix="back" x_pos="-0.12"/>
+  </xacro:macro> -->
 </robot>

File: xacro/laser_scanner.xacro (robot description, xacro)
@@ -75,5 +75,5 @@
                 <plugin name="gazebo_ros_laser_" filename="libgazebo_ros_ray_sensor.so">
                     <topicName>/scan</topicName>
-                    <!-- <output_type>sensor_msgs/LaserScan</output_type> -->
+                    <output_type>sensor_msgs/LaserScan</output_type>
                     <ros>
                         <!-- <namespace>/${robot_name}</namespace> -->

Commit message: initial changes to launch file and xacro to reflect in progress

File: xacro/barista_robot_model.urdf.xacro (robot description, xacro)
@@ -3,7 +3,7 @@
     <!-- Declare arguments -->
     <!-- <xacro:arg name="robot_name" default="barista_robot"/> -->
-    <xacro:arg name="colour" default="Gazebo/Blue"/>
+    <!-- <xacro:arg name="colour" default="Gazebo/Blue"/> -->
     <!-- Create properties from arguments -->
-    <!-- <xacro:property name="robot_name" value="$(arg robot_name)"/> -->
+    <xacro:property name="robot_name" value="$(arg robot_name)"/>
     <xacro:property name="colour" value="$(arg colour)"/>
     <xacro:arg name="include_laser" default="true"/>

Commit message: spawn rick and morty in both gazebo and rviz without tf and frames conflict. correction in colour for rviz and collision for standoff rods

File: xacro/barista_robot_model.urdf.xacro (robot description, xacro)
@@ -1,7 +1,8 @@
 <?xml version="1.0"?>
-<robot xmlns:xacro="http://www.ros.org/wiki/xacro" name="barista_robot">
-    <!-- Declare arguments -->
-    <!-- <xacro:arg name="robot_name" default="barista_robot"/> -->
-    <!-- <xacro:arg name="colour" default="Gazebo/Blue"/> -->
+<!-- <robot xmlns:xacro="http://www.ros.org/wiki/xacro" name="barista_robot"> -->
+<robot xmlns:xacro="http://www.ros.org/wiki/xacro" name="$(arg robot_name)">
+    <!-- Accept arguments from launch file -->
+    <xacro:arg name="robot_name" default="barista_robot"/>
+    <xacro:arg name="colour" default="Gazebo/Black"/>
     <!-- Create properties from arguments -->
     <xacro:property name="robot_name" value="$(arg robot_name)"/>
@@ -29,4 +30,5 @@
         <color rgba="1.0 1.0 1.0 1"/>
     </material>
+    <!-- <link name="${robot_name}/base_link"> -->
     <link name="base_link">
         <inertial>
@@ -37,4 +39,5 @@
     </link>
     <!-- chassis -->
+    <!-- <link name="${robot_name}/chassis"> -->
     <link name="chassis">
         <visual>
@@ -42,5 +45,13 @@
                 <cylinder length="0.155" radius="0.178"/>
             </geometry>
-            <material name="blue"/>
+            <!-- <material name="blue"/> -->
+            <material name="${robot_name}_material">
+                <xacro:if value="${robot_name == 'rick'}">
+                    <color rgba="0.0 0.0 1.0 1.0"/>  <!-- Blue -->
+                </xacro:if>
+                <xacro:if value="${robot_name == 'morty'}">
+                    <color rgba="1.0 0.0 0.0 1.0"/>  <!-- Red -->
+                </xacro:if>
+            </material>
         </visual>
         <collision>
@@ -68,32 +79,33 @@
     <!-- Drive Wheel -->
     <xacro:include filename="$(find barista_robot_description)/xacro/drive_wheel.xacro"/>
-    <xacro:drive_wheel prefix="left" reflect="1"/>
-    <xacro:drive_wheel prefix="right" reflect="-1"/>
+    <xacro:drive_wheel prefix="left" reflect="1" robot_name="${robot_name}"/>
+    <xacro:drive_wheel prefix="right" reflect="-1" robot_name="${robot_name}"/>
     <!-- Standoff Post -->
     <xacro:include filename="$(find barista_robot_description)/xacro/standoff_rod.xacro"/>
-    <xacro:standoff_rod prefix="front_left" rod_radius="0.010" rod_height="0.220" x_reflect="1" y_reflect="1"/>
-    <xacro:standoff_rod prefix="front_right" rod_radius="0.010" rod_height="0.220" x_reflect="1" y_reflect="-1"/>
-    <xacro:standoff_rod prefix="back_left" rod_radius="0.010" rod_height="0.220" x_reflect="-1" y_reflect="1"/>
-    <xacro:standoff_rod prefix="back_right" rod_radius="0.010" rod_height="0.220" x_reflect="-1" y_reflect="-1"/>
+    <xacro:standoff_rod prefix="front_left" rod_radius="0.010" rod_height="0.220" x_reflect="1" y_reflect="1" robot_name="${robot_name}"/>
+    <xacro:standoff_rod prefix="front_right" rod_radius="0.010" rod_height="0.220" x_reflect="1" y_reflect="-1" robot_name="${robot_name}"/>
+    <xacro:standoff_rod prefix="back_left" rod_radius="0.010" rod_height="0.220" x_reflect="-1" y_reflect="1" robot_name="${robot_name}"/>
+    <xacro:standoff_rod prefix="back_right" rod_radius="0.010" rod_height="0.220" x_reflect="-1" y_reflect="-1" robot_name="${robot_name}"/>
     <!-- Caster Wheels -->
     <xacro:include filename="$(find barista_robot_description)/xacro/caster_wheel.xacro"/>
-    <xacro:caster_wheel prefix="front" x_pos="0.12"/>
-    <xacro:caster_wheel prefix="back" x_pos="-0.12"/>
+    <xacro:caster_wheel prefix="front" x_pos="0.12" robot_name="${robot_name}"/>
+    <xacro:caster_wheel prefix="back" x_pos="-0.12" robot_name="${robot_name}"/>
     <!-- Cup Holder Tray -->
     <xacro:include filename="$(find barista_robot_description)/xacro/cup_holder_tray.xacro"/>
     <!-- <xacro:cup_holder_tray colour="Gazebo/Blue" /> -->
-    <xacro:cup_holder_tray colour="${colour}" />
+            <!-- <material name="${robot_name}_colour"/> -->
+    <xacro:cup_holder_tray colour="${colour}" robot_name="${robot_name}"/>
     <!-- Laser Scanner -->
     <xacro:include filename="$(find barista_robot_description)/xacro/laser_scanner.xacro"/>
     <!-- Include laser with default behavior -->
-    <!-- <xacro:laser_scanner include_laser="true" robot_name="$(arg robot_name)"/> -->
-    <xacro:laser_scanner include_laser="$(arg include_laser)" />
-    <!-- <xacro:laser_scanner include_laser="true" /> -->
+    <xacro:laser_scanner include_laser="true" robot_name="${robot_name}"/>
+    <!-- <xacro:laser_scanner include_laser="$(arg include_laser)" /> -->
     <!-- libgazebo_ros_joint_state_publisher -->
     <gazebo>
-        <plugin name="barista_robot_joint_state" filename="libgazebo_ros_joint_state_publisher.so">
+        <!-- <plugin name="barista_robot_joint_state" filename="libgazebo_ros_joint_state_publisher.so"> -->
+        <plugin name="${robot_name}_joint_state" filename="libgazebo_ros_joint_state_publisher.so">
         <ros>
             <!-- <namespace>/${robot_name}</namespace> -->
-            <!-- <namespace>/</namespace> -->
+            <namespace>${robot_name}</namespace>
             <remapping>~/out:=joint_states</remapping>
         </ros>
@@ -112,9 +124,10 @@
     <gazebo>
         <plugin filename="libgazebo_ros_diff_drive.so" name="differential_drive_controller">
-            <!-- <ros>
-                <namespace>/${robot_name}</namespace>
-                <namespace>/</namespace>
+            <ros>
+                <!-- <namespace>/${robot_name}</namespace>
+                <remapping>/cmd_vel:=cmd_vel</remapping> -->
+                <namespace>${robot_name}</namespace>
                 <remapping>/cmd_vel:=cmd_vel</remapping>
-            </ros> -->
+            </ros>
             <update_rate>30</update_rate>
             <!-- wheels -->
@@ -129,12 +142,12 @@
             <max_wheel_acceleration>2.0</max_wheel_acceleration>
             <!-- Receive velocity commands on this ROS topic -->
-            <command_topic>cmd_vel</command_topic>
+            <!-- <command_topic>cmd_vel</command_topic> -->
             <!-- output -->
             <publish_odom>true</publish_odom>
             <publish_odom_tf>true</publish_odom_tf>
-            <!-- <odometry_frame>${robot_name}/odom</odometry_frame>
-            <robot_base_frame>${robot_name}/base_link</robot_base_frame> -->
-            <odometry_frame>odom</odometry_frame>
-            <robot_base_frame>base_link</robot_base_frame>
+            <odometry_frame>${robot_name}/odom</odometry_frame>
+            <robot_base_frame>${robot_name}/base_link</robot_base_frame>
+            <!-- <odometry_frame>odom</odometry_frame>
+            <robot_base_frame>base_link</robot_base_frame> -->
             <!-- Odometry source, 0 for ENCODER, 1 for WORLD, defaults to WORLD -->
             <odometry_source>1</odometry_source>

File: xacro/caster_wheel.xacro (robot description, xacro)
@@ -2,5 +2,5 @@
 <robot xmlns:xacro="http://www.ros.org/wiki/xacro">
   <!-- Caster wheel macro -->
-  <xacro:macro name="caster_wheel" params="prefix x_pos">
+  <xacro:macro name="caster_wheel" params="prefix x_pos robot_name">
     <!-- Properties -->
     <xacro:property name="wheel_radius" value="0.0352"/>
@@ -8,4 +8,5 @@
     <xacro:property name="wheel_mass" value="0.1"/>
     <!-- Yaw link -->
+    <!-- <link name="${robot_name}/${prefix}_yaw_link"> -->
     <link name="${prefix}_yaw_link">
         <visual>
@@ -27,6 +28,8 @@
         </inertial>
     </link>
-    <joint name="${prefix}_yaw_joint" type="fixed">
+    <joint name="${robot_name}/${prefix}_yaw_joint" type="fixed">
         <origin rpy="0 1.5707 1.5707" xyz="${x_pos} 0.0 -0.070" />
+        <!-- <parent link="${robot_name}/chassis" />
+        <child link="${robot_name}/${prefix}_yaw_link" /> -->
         <parent link="chassis" />
         <child link="${prefix}_yaw_link" />
@@ -103,8 +106,3 @@
     </gazebo>
   </xacro:macro>
-  <!-- Need to check this way of implementation too -->
-  <!-- <xacro:macro name="caster_wheel">
-    <xacro:caster_wheel prefix="front" x_pos="0.12"/>
-    <xacro:caster_wheel prefix="back" x_pos="-0.12"/>
-  </xacro:macro> -->
 </robot>

File: xacro/cup_holder_tray.xacro (robot description, xacro)
@@ -2,5 +2,15 @@
 <robot xmlns:xacro="http://www.ros.org/wiki/xacro">
   <!-- Cupholder tray macro -->
-  <xacro:macro name="cup_holder_tray" params="colour">
+  <xacro:macro name="cup_holder_tray" params="colour robot_name">
+    <xacro:if value="${robot_name == 'rick'}">
+        <material name="sep_colour">
+            <color rgba="0.0 0.0 1.0 1.0"/> <!--  Blue -->
+        </material>
+    </xacro:if>
+    <xacro:if value="${robot_name == 'morty'}">
+        <material name="sep_colour">
+            <color rgba="1.0 0.0 0.0 1.0"/> <!--  Red -->
+        </material>
+    </xacro:if>
     <!-- Xacro properties for wheel dimensions -->
     <xacro:property name="tray_radius" value="0.160"/>
@@ -11,5 +21,13 @@
                 <cylinder length="${tray_height}" radius="${tray_radius}"/>
             </geometry>
-            <material name="blue"/>
+            <!-- <material name="blue"/> -->
+            <material name="${robot_name}_material">
+                <xacro:if value="${robot_name == 'rick'}">
+                    <color rgba="0.0 0.0 1.0 1.0"/>  <!-- Blue -->
+                </xacro:if>
+                <xacro:if value="${robot_name == 'morty'}">
+                    <color rgba="1.0 0.0 0.0 1.0"/>  <!-- Red -->
+                </xacro:if>
+            </material>
         </visual>
         <collision>

File: xacro/drive_wheel.xacro (robot description, xacro)
@@ -2,5 +2,5 @@
 <robot xmlns:xacro="http://www.ros.org/wiki/xacro">
   <!-- Drive wheel macro -->
-  <xacro:macro name="drive_wheel" params="prefix reflect">
+  <xacro:macro name="drive_wheel" params="prefix reflect robot_name">
     <!-- Xacro properties for wheel dimensions -->
     <xacro:property name="wheel_radius" value="0.0352"/>

File: xacro/laser_scanner.xacro (robot description, xacro)
@@ -2,6 +2,5 @@
 <robot xmlns:xacro="http://www.ros.org/wiki/xacro">
     <!-- Laser Scanner macro -->
-    <!-- <xacro:macro name="laser_scanner" params="include_laser robot_name"> -->
-    <xacro:macro name="laser_scanner" params="include_laser">
+    <xacro:macro name="laser_scanner" params="include_laser robot_name">
     <!-- Only create laser if include_laser is true -->
     <xacro:if value="${include_laser}">
@@ -42,6 +41,5 @@
         <!-- Gazebo Laser Scanner Plugin -->
         <gazebo reference="laser_optical_frame">
-            <!-- <sensor type="ray" name="laser_scanner_${robot_name}"> -->
-            <sensor type="ray" name="laser_scanner">
+            <sensor type="ray" name="${robot_name}_laser_scanner">
                 <pose>0 0 0 0 0 0</pose>
                 <update_rate>10</update_rate>
@@ -72,14 +70,11 @@
                 <always_on>true</always_on>
                 <visualize>true</visualize>
-                <!-- <plugin name="gazebo_ros_laser_${robot_name}" filename="libgazebo_ros_ray_sensor.so"> -->
-                <plugin name="gazebo_ros_laser_" filename="libgazebo_ros_ray_sensor.so">
-                    <topicName>/scan</topicName>
+                <plugin name="${robot_name}_gazebo_ros_laser" filename="libgazebo_ros_ray_sensor.so">
                     <output_type>sensor_msgs/LaserScan</output_type>
                     <ros>
-                        <!-- <namespace>/${robot_name}</namespace> -->
-                        <namespace>/</namespace>
+                        <namespace>/${robot_name}</namespace>
                         <remapping>~/out:=scan</remapping>
                     </ros>
-                <frame_name>laser_optical_frame</frame_name>
+                    <frame_name>${robot_name}/laser_optical_frame</frame_name>
                 </plugin>
             </sensor>

File: xacro/standoff_rod.xacro (robot description, xacro)
@@ -2,5 +2,5 @@
 <robot xmlns:xacro="http://www.ros.org/wiki/xacro">
   <!-- Standoff post macro -->
-  <xacro:macro name="standoff_rod" params="prefix rod_radius rod_height x_reflect y_reflect">
+  <xacro:macro name="standoff_rod" params="prefix rod_radius rod_height x_reflect y_reflect robot_name">
     <!-- Xacro properties for wheel dimensions -->
     <xacro:property name="x_pos" value="0.065"/>
@@ -20,5 +20,5 @@
         <collision>
             <geometry>
-                <cylinder length="${rod_radius}" radius="${rod_height}"/>
+                <cylinder radius="${rod_radius}" length="${rod_height}"/>
             </geometry>
         </collision>
