Commit message: Including physics property.yaml file for rapid testing

File: xacro/barista_robot_model.urdf.xacro (robot description, xacro)
@@ -2,4 +2,6 @@
 <!-- <robot xmlns:xacro="http://www.ros.org/wiki/xacro" name="barista_robot"> -->
 <robot xmlns:xacro="http://www.ros.org/wiki/xacro" name="$(arg robot_name)">
+    <!-- Load physics parameters -->
+    <xacro:include filename="$(find barista_robot_description)/xacro/physics_properties.xacro"/>
     <!-- Accept arguments from launch file -->
     <xacro:arg name="robot_name" default="barista_robot"/>
@@ -30,18 +32,25 @@
         <color rgba="1.0 1.0 1.0 1"/>
     </material>
-    <!-- <link name="${robot_name}/base_link"> -->
+    <xacro:property name="base_width" value="0.356"/>
+    <xacro:property name="base_height" value="0.155"/>
     <link name="base_link">
         <inertial>
             <origin xyz="0 0 0.5" rpy="0 0 0"/>
-            <mass value="1.0"/>
-            <inertia ixx="0.01" ixy="0" ixz="0" iyy="0.01" iyz="0" izz="0.01"/>
+            <!-- <mass value="2.0"/>
+            <inertia ixx="0.008" ixy="0" ixz="0"
+                    iyy="0.008" iyz="0"
+                    izz="0.012"/> -->
+            <mass value="${physics_config['base_mass']}"/>
+            <inertia ixx="${physics_config['base_mass'] * physics_config['base_ixx_factor']}"
+                     iyy="${physics_config['base_mass'] * physics_config['base_iyy_factor']}"
+                     izz="${physics_config['base_mass'] * physics_config['base_izz_factor']}"
+                     ixy="0" ixz="0" iyz="0"/>
         </inertial>
     </link>
     <!-- chassis -->
-    <!-- <link name="${robot_name}/chassis"> -->
     <link name="chassis">
         <visual>
             <geometry>
-                <cylinder length="0.155" radius="0.178"/>
+                <cylinder length="${base_height}" radius="${base_width/2}"/>
             </geometry>
             <!-- <material name="blue"/> -->
@@ -57,12 +66,12 @@
         <collision>
             <geometry>
-                <cylinder length="0.155" radius="0.178"/>
+                <cylinder length="${base_height}" radius="${base_width/2}"/>
             </geometry>
         </collision>
         <inertial>
-            <origin xyz="0 0 0" rpy="0 0 0"/>
-            <mass value="0.8"/>
-            <!-- <inertia ixx="0.1" ixy="0" ixz="0" iyy="0.1" iyz="0" izz="0.15"/> -->
-            <inertia ixx="0.007938466666666666" ixy="0" ixz="0" iyy="0.007938466666666666" iyz="0" izz="0.0126736"/>
+            <mass value="0.5"/>
+            <inertia ixx="0.002" ixy="0" ixz="0"
+                    iyy="0.002" iyz="0"
+                    izz="0.003"/>
         </inertial>
     </link>
@@ -71,6 +80,4 @@
         <parent link="base_link"/>
         <child link="chassis"/>
-        <axis xyz="0.0 0.0 0.0"/>
-        <limit lower="0.0" upper="0.0" effort="0.0" velocity="0.0"/>
     </joint>
     <gazebo reference="chassis">
@@ -93,6 +100,4 @@
     <!-- Cup Holder Tray -->
     <xacro:include filename="$(find barista_robot_description)/xacro/cup_holder_tray.xacro"/>
-    <!-- <xacro:cup_holder_tray colour="Gazebo/Blue" /> -->
-            <!-- <material name="${robot_name}_colour"/> -->
     <xacro:cup_holder_tray colour="${colour}" robot_name="${robot_name}"/>
     <!-- Laser Scanner -->
@@ -100,11 +105,8 @@
     <!-- Include laser with default behavior -->
     <xacro:laser_scanner include_laser="true" robot_name="${robot_name}"/>
-    <!-- <xacro:laser_scanner include_laser="$(arg include_laser)" /> -->
     <!-- libgazebo_ros_joint_state_publisher -->
     <gazebo>
-        <!-- <plugin name="barista_robot_joint_state" filename="libgazebo_ros_joint_state_publisher.so"> -->
         <plugin name="${robot_name}_joint_state" filename="libgazebo_ros_joint_state_publisher.so">
         <ros>
-            <!-- <namespace>/${robot_name}</namespace> -->
             <namespace>${robot_name}</namespace>
             <remapping>~/out:=joint_states</remapping>
@@ -125,12 +127,9 @@
         <plugin filename="libgazebo_ros_diff_drive.so" name="differential_drive_controller">
             <ros>
-                <!-- <namespace>/${robot_name}</namespace>
-                <remapping>/cmd_vel:=cmd_vel</remapping> -->
                 <namespace>${robot_name}</namespace>
                 <remapping>/cmd_vel:=cmd_vel</remapping>
             </ros>
-            <update_rate>30</update_rate>
+            <update_rate>60</update_rate>
             <!-- wheels -->
-            <!-- <num_wheel_pairs>1</num_wheel_pairs> -->
             <left_joint>joint_left_wheel</left_joint>
             <right_joint>joint_right_wheel</right_joint>
@@ -139,6 +138,6 @@
             <wheel_diameter>0.0704</wheel_diameter>
             <!-- limits -->
-            <max_wheel_torque>1.0</max_wheel_torque>
-            <max_wheel_acceleration>2.0</max_wheel_acceleration>
+            <max_wheel_torque>1.5</max_wheel_torque>       <!-- Much lower -->
+            <max_wheel_acceleration>0.3</max_wheel_acceleration>  <!-- Gentler -->
             <!-- Receive velocity commands on this ROS topic -->
             <!-- <command_topic>cmd_vel</command_topic> -->
@@ -146,12 +145,8 @@
             <publish_odom>true</publish_odom>
             <publish_odom_tf>true</publish_odom_tf>
+            <!-- try to remove this later -->
+            <publish_wheel_tf>false</publish_wheel_tf>
             <odometry_frame>${robot_name}/odom</odometry_frame>
             <robot_base_frame>${robot_name}/base_link</robot_base_frame>
-            <!-- <odometry_frame>odom</odometry_frame>
-            <robot_base_frame>base_link</robot_base_frame> -->
-            <!-- Odometry source, 0 for ENCODER, 1 for WORLD, defaults to WORLD -->
-            <odometry_source>1</odometry_source>
-            <!-- Set to true to publish transforms for the wheel links. -->
-            <!-- <publish_wheel_tf>true</publish_wheel_tf> -->
         </plugin>
     </gazebo>

File: xacro/caster_wheel.xacro (robot description, xacro)
@@ -6,7 +6,8 @@
     <xacro:property name="wheel_radius" value="0.0352"/>
     <xacro:property name="cylinder_length" value="0.010"/>
-    <xacro:property name="wheel_mass" value="0.1"/>
+    <xacro:property name="wheel_mass" value="0.02"/>
+    <xacro:property name="joint_type" value="fixed"/>
+    <!-- <xacro:property name="joint_type" value="continuous"/> -->
     <!-- Yaw link -->
-    <!-- <link name="${robot_name}/${prefix}_yaw_link"> -->
     <link name="${prefix}_yaw_link">
         <visual>
@@ -23,18 +24,16 @@
         <inertial>
             <mass value="${wheel_mass}"/>
-            <inertia ixx="3.1809333333333334e-05" ixy="0" ixz="0"
-                     iyy="3.1809333333333334e-05" iyz="0"
-                     izz="6.1952e-05"/>
+            <inertia ixx="0.0000031184" ixy="0" ixz="0" iyy="0.0000031184" iyz="0" izz="0.000006195"/>
         </inertial>
     </link>
-    <joint name="${robot_name}/${prefix}_yaw_joint" type="fixed">
+    <joint name="${robot_name}/${prefix}_yaw_joint" type="${joint_type}">
         <origin rpy="0 1.5707 1.5707" xyz="${x_pos} 0.0 -0.070" />
-        <!-- <parent link="${robot_name}/chassis" />
-        <child link="${robot_name}/${prefix}_yaw_link" /> -->
         <parent link="chassis" />
         <child link="${prefix}_yaw_link" />
-        <axis xyz="0 1 0" />
+        <!-- <axis xyz="0 1 0" /> -->
+        <axis xyz="0 0 1 " />
         <limit effort="1000.0" velocity="100.0" />
-        <dynamics damping="0.5" friction="0.5"/>
+        <!-- <dynamics damping="2.0" friction="0.5"/> -->
+        <dynamics damping="3.0" friction="0.7"/>
     </joint>
     <!-- Roll link -->
@@ -53,16 +52,17 @@
         <inertial>
             <mass value="${wheel_mass}"/>
-            <inertia ixx="3.1809333333333334e-05" ixy="0" ixz="0"
-                     iyy="3.1809333333333334e-05" iyz="0"
-                     izz="6.1952e-05"/>
+            <inertia ixx="0.0000031184" ixy="0" ixz="0" iyy="0.0000031184" iyz="0" izz="0.000006195"/>
         </inertial>
     </link>
-    <joint name="${prefix}_roll_joint" type="fixed">
-        <origin rpy="0 1.5707 1.5707" xyz="0 0 0" />
+    <joint name="${prefix}_roll_joint" type="${joint_type}">
+        <!-- <origin rpy="0 1.5707 1.5707" xyz="0 0 0" /> -->
+        <origin rpy="0 0 0" xyz="0 0 0" />
         <parent link="${prefix}_yaw_link" />
         <child link="${prefix}_roll_link" />
-        <axis xyz="1 0 0" />
+        <!-- <axis xyz="1 0 0" /> -->
+        <axis xyz="0 1 0" />
         <limit effort="1000.0" velocity="100.0" />
-        <dynamics damping="0.5" friction="0.5"/>
+        <!-- <dynamics damping="0.5" friction="0.1"/> -->
+        <dynamics damping="1.0" friction="0.5"/>
     </joint>
     <!-- Pitch link -->
@@ -80,28 +80,84 @@
         </collision>
         <inertial>
-            <origin xyz="0 0 0" rpy="0 0 0"/>
             <mass value="${wheel_mass}"/>
-            <inertia ixx="4.95616e-05" ixy="0" ixz="0"
-                     iyy="4.95616e-05" iyz="0"
-                     izz="4.95616e-05"/>
+            <inertia ixx="0.00000826" ixy="0" ixz="0"
+                     iyy="00.00000826" iyz="0"
+                     izz="0.00000826"/>
         </inertial>
     </link>
-    <joint name="${prefix}_pitch_joint" type="fixed">
-        <origin rpy="0 1.5707 1.5707" xyz="0 0 0" />
+    <joint name="${prefix}_pitch_joint" type="${joint_type}">
+        <!-- <origin rpy="0 1.5707 1.5707" xyz="0 0 0" /> -->
+        <origin rpy="0 0 0" xyz="0 0 0" />
         <parent link="${prefix}_roll_link" />
         <child link="${prefix}_pitch_link" />
-        <axis xyz="0 1 0" />
+        <!-- <axis xyz="0 1 0" /> -->
+        <!-- <axis xyz="0 0 1" /> -->
+        <!-- <axis xyz="1 0 0" /> -->
         <limit effort="1000.0" velocity="100.0" />
-        <dynamics damping="0.5" friction="0.5"/>
+        <dynamics damping="0.01" friction="0.01"/>
     </joint>
     <!-- Gazebo materials -->
     <gazebo reference="${prefix}_yaw_link">
         <material>Gazebo/Grey</material>
+        <surface>
+            <friction>
+                <ode>
+                    <mu>0.01</mu>
+                    <mu2>0.01</mu2>
+                    <slip1>0.9</slip1>
+                    <slip2>0.9</slip2>
+                </ode>
+            </friction>
+            <contact>
+                <ode>
+                    <kp>100.0</kp>
+                    <kd>1.0</kd>
+                    <soft_cfm>0.01</soft_cfm>
+                    <soft_erp>0.2</soft_erp>
+                </ode>
+            </contact>
+        </surface>
     </gazebo>
     <gazebo reference="${prefix}_roll_link">
         <material>Gazebo/Grey</material>
+        <surface>
+            <friction>
+                <ode>
+                    <mu>0.01</mu>
+                    <mu2>0.01</mu2>
+                    <slip1>0.5</slip1>
+                    <slip2>0.5</slip2>
+                </ode>
+            </friction>
+            <contact>
+                <ode>
+                    <kp>100.0</kp>
+                    <kd>1.0</kd>
+                    <soft_cfm>0.01</soft_cfm>
+                    <soft_erp>0.2</soft_erp>
+                </ode>
+            </contact>
+        </surface>
     </gazebo>
     <gazebo reference="${prefix}_pitch_link">
         <material>Gazebo/Grey</material>
+        <surface>
+            <friction>
+                <ode>
+                    <mu>0.01</mu>
+                    <mu2>0.01</mu2>
+                    <slip1>0.5</slip1>
+                    <slip2>0.5</slip2>
+                </ode>
+            </friction>
+            <contact>
+                <ode>
+                    <kp>100.0</kp>
+                    <kd>1.0</kd>
+                    <soft_cfm>0.01</soft_cfm>
+                    <soft_erp>0.2</soft_erp>
+                </ode>
+            </contact>
+        </surface>
     </gazebo>
   </xacro:macro>

File: xacro/cup_holder_tray.xacro (robot description, xacro)
@@ -37,6 +37,6 @@
         </collision>
         <inertial>
-            <mass value="1.0"/>
-            <inertia ixx="0.007075" ixy="0" ixz="0" iyy="0.007075" iyz="0" izz="0.0128"/>
+            <mass value="0.02"/>
+            <inertia ixx="0.00008117" ixy="0" ixz="0" iyy="0.00008117" iyz="0" izz="0.000001"/>
         </inertial>
     </link>

File: xacro/drive_wheel.xacro (robot description, xacro)
@@ -1,6 +1,8 @@
 <?xml version="1.0"?>
 <robot xmlns:xacro="http://www.ros.org/wiki/xacro">
-  <!-- Drive wheel macro -->
-  <xacro:macro name="drive_wheel" params="prefix reflect robot_name">
+    <!-- Load physics parameters -->
+    <xacro:include filename="$(find barista_robot_description)/xacro/physics_properties.xacro"/>
+    <!-- Drive wheel macro -->
+    <xacro:macro name="drive_wheel" params="prefix reflect robot_name">
     <!-- Xacro properties for wheel dimensions -->
     <xacro:property name="wheel_radius" value="0.0352"/>
@@ -11,5 +13,5 @@
                 <cylinder length="${wheel_width}" radius="${wheel_radius}"/>
             </geometry>
-            <material name="red"/>
+            <material name="black"/>
         </visual>
         <collision>
@@ -19,12 +21,37 @@
         </collision>
         <inertial>
-            <mass value="0.07"/>
-            <inertia ixx="2.4158633333333336e-05" ixy="0" ixz="0"
-                     iyy="2.4158633333333336e-05" iyz="0"
-                     izz="4.3366400000000005e-05"/>
+            <!-- <mass value="0.05"/>
+            <inertia ixx="0.000005752" ixy="0" ixz="0"
+                    iyy="0.000005752" iyz="0"
+                    izz="0.000010325"/> -->
+            <mass value="${physics_config['wheel_mass']}"/>
+            <inertia ixx="${physics_config['wheel_mass'] * physics_config['wheel_ixx_factor']}"
+                    iyy="${physics_config['wheel_mass'] * physics_config['wheel_iyy_factor']}"
+                    izz="${physics_config['wheel_mass'] * physics_config['wheel_izz_factor']}"
+                    ixy="0" ixz="0" iyz="0"/>
         </inertial>
     </link>
     <gazebo reference="${prefix}_wheel">
         <material>Gazebo/Black</material>
+        <surface>
+            <friction>
+                <ode>
+                    <mu>1.5</mu>
+                    <mu2>1.5</mu2>
+                    <slip1>0.01</slip1>
+                    <slip2>0.01</slip2>
+                </ode>
+            </friction>
+            <contact>
+                <ode>
+                    <kp>1000.0</kp>
+                    <kd>1.0</kd>
+                    <soft_cfm>0.0</soft_cfm>
+                    <soft_erp>0.2</soft_erp>
+                    <max_vel>0.01</max_vel>
+                    <min_depth>0.001</min_depth>
+                </ode>
+            </contact>
+        </surface>
     </gazebo>
     <joint name="joint_${prefix}_wheel" type="continuous">
@@ -32,7 +59,9 @@
         <child link="${prefix}_wheel"/>
         <parent link="chassis"/>
-        <axis rpy="0 0 0" xyz="0 1 0"/>
+        <axis rpy="0 0 0" xyz="0 0 1"/>
         <limit effort="10000" velocity="1000"/>
-        <joint_properties damping="0.5" friction="0.5"/>
+        <!-- <joint_properties damping="3.0" friction="0.4"/> -->
+    <joint_properties damping="${physics_config['wheel_damping']}"
+                     friction="${physics_config['wheel_friction']}"/>
     </joint>
   </xacro:macro>

File: xacro/laser_scanner.xacro (robot description, xacro)
@@ -18,6 +18,8 @@
             </collision>
             <inertial>
-                <mass value="0.3"/>
-                <inertia ixx="0.001" ixy="0" ixz="0" iyy="0.001" iyz="0" izz="0.0005"/>
+                <!-- <mass value="0.3"/>
+                <inertia ixx="0.001" ixy="0" ixz="0" iyy="0.001" iyz="0" izz="0.0005"/> -->
+                <mass value="0.01"/>
+                <inertia ixx="6.066578520833334e-06" ixy="0" ixz="0" iyy="6.072950163333333e-06" iyz="0" izz="9.365128684166666e-06"/>
             </inertial>
         </link>
@@ -44,8 +46,10 @@
                 <pose>0 0 0 0 0 0</pose>
                 <update_rate>10</update_rate>
+                <always_on>true</always_on>
+                <visualize>true</visualize>
                 <ray>
                     <scan>
                         <horizontal>
-                            <samples>360</samples>
+                            <samples>200</samples>
                             <resolution>1</resolution>
                             <min_angle>-3.14159</min_angle>
@@ -68,6 +72,4 @@
                     </noise>
                 </ray>
-                <always_on>true</always_on>
-                <visualize>true</visualize>
                 <plugin name="${robot_name}_gazebo_ros_laser" filename="libgazebo_ros_ray_sensor.so">
                     <output_type>sensor_msgs/LaserScan</output_type>

File: xacro/standoff_rod.xacro (robot description, xacro)
@@ -15,6 +15,8 @@
         </visual>
         <inertial>
-            <mass value="0.1"/>
-            <inertia ixx="0.00040583333333333335" ixy="0" ixz="0" iyy="0.00040583333333333335" iyz="0" izz="5e-06"/>
+            <mass value="0.02"/>
+            <inertia ixx="0.00008117" ixy="0" ixz="0"
+                     iyy="0.00008117" iyz="0"
+                     izz="0.000001"/>
         </inertial>
         <collision>
