Commit message: changes related to all continious joints to accept physics property xacro file

File: xacro/barista_robot_model.urdf.xacro (robot description, xacro)
@@ -35,16 +35,4 @@
     <xacro:property name="base_height" value="0.155"/>
     <link name="base_link">
-        <inertial>
-            <origin xyz="0 0 0.5" rpy="0 0 0"/>
-            <!-- <mass value="2.0"/>
-            <inertia ixx="0.008" ixy="0" ixz="0"
-                    iyy="0.008" iyz="0"
-                    izz="0.012"/> -->
-            <mass value="${physics_config['base_mass']}"/>
-            <inertia ixx="${physics_config['base_mass'] * physics_config['base_ixx_factor']}"
-                     iyy="${physics_config['base_mass'] * physics_config['base_iyy_factor']}"
-                     izz="${physics_config['base_mass'] * physics_config['base_izz_factor']}"
-                     ixy="0" ixz="0" iyz="0"/>
-        </inertial>
     </link>
     <!-- chassis -->
@@ -112,5 +100,5 @@
             <remapping>~/out:=joint_states</remapping>
         </ros>
-        <update_rate>30</update_rate>
+        <update_rate>${physics_config['jsp_update_rate']}</update_rate>
         <joint_name>joint_left_wheel</joint_name>
         <joint_name>joint_right_wheel</joint_name>
@@ -130,5 +118,5 @@
                 <remapping>/cmd_vel:=cmd_vel</remapping>
             </ros>
-            <update_rate>60</update_rate>
+            <update_rate>${physics_config['diff_update_rate']}</update_rate>
             <!-- wheels -->
             <left_joint>joint_left_wheel</left_joint>
@@ -138,8 +126,8 @@
             <wheel_diameter>0.0704</wheel_diameter>
             <!-- limits -->
-            <max_wheel_torque>1.5</max_wheel_torque>       <!-- Much lower -->
-            <max_wheel_acceleration>0.3</max_wheel_acceleration>  <!-- Gentler -->
-            <!-- Receive velocity commands on this ROS topic -->
-            <!-- <command_topic>cmd_vel</command_topic> -->
+            <max_wheel_torque>${physics_config['max_wheel_torque']}</max_wheel_torque>
+            <max_wheel_acceleration>${physics_config['max_wheel_acceleration']}</max_wheel_acceleration>
+            <max_linear_velocity>${physics_config['max_linear_velocity']}</max_linear_velocity>
+            <max_angular_velocity>${physics_config['max_angular_velocity']}</max_angular_velocity>
             <!-- output -->
             <publish_odom>true</publish_odom>

File: xacro/caster_wheel.xacro (robot description, xacro)
@@ -9,6 +9,6 @@
     <xacro:property name="cylinder_length" value="0.010"/>
     <xacro:property name="wheel_mass" value="0.02"/>
-    <xacro:property name="joint_type" value="fixed"/>
-    <!-- <xacro:property name="joint_type" value="continuous"/> -->
+    <!-- <xacro:property name="joint_type" value="fixed"/> -->
+    <xacro:property name="joint_type" value="continuous"/>
     <!-- Yaw link -->
     <link name="${prefix}_yaw_link">
@@ -25,6 +25,4 @@
         </collision>
         <inertial>
-            <!-- <mass value="${wheel_mass}"/>
-            <inertia ixx="0.0000031184" ixy="0" ixz="0" iyy="0.0000031184" iyz="0" izz="0.000006195"/> -->
             <mass value="${physics_config['caster_mass']}"/>
             <inertia ixx="${physics_config['caster_yr_ixx']}" ixy="0" ixz="0"
@@ -40,7 +38,6 @@
         <axis xyz="0 0 1 " />
         <limit effort="1000.0" velocity="100.0" />
-        <!-- <dynamics damping="3.0" friction="0.7"/> -->
-        <dynamics damping="${physics_config['wheel_damping']}"
-                        friction="${physics_config['wheel_friction']}"/>
+        <dynamics damping="${physics_config['caster_damping']}"
+                        friction="${physics_config['caster_friction']}"/>
     </joint>
     <!-- Roll link -->
@@ -58,6 +55,4 @@
         </collision>
         <inertial>
-            <!-- <mass value="${wheel_mass}"/>
-            <inertia ixx="0.0000031184" ixy="0" ixz="0" iyy="0.0000031184" iyz="0" izz="0.000006195"/> -->
             <mass value="${physics_config['caster_mass']}"/>
             <inertia ixx="${physics_config['caster_yr_ixx']}" ixy="0" ixz="0"
@@ -67,5 +62,4 @@
     </link>
     <joint name="${prefix}_roll_joint" type="${joint_type}">
-        <!-- <origin rpy="0 1.5707 1.5707" xyz="0 0 0" /> -->
         <origin rpy="0 1.5707 1.5707" xyz="0 0 0" />
         <parent link="${prefix}_yaw_link" />
@@ -74,7 +68,6 @@
         <axis xyz="0 1 0" />
         <limit effort="1000.0" velocity="100.0" />
-        <!-- <dynamics damping="1.0" friction="0.5"/> -->
-        <dynamics damping="${physics_config['wheel_damping']}"
-                        friction="${physics_config['wheel_friction']}"/>
+        <dynamics damping="${physics_config['caster_damping']}"
+                        friction="${physics_config['caster_friction']}"/>
     </joint>
     <!-- Pitch link -->
@@ -92,8 +85,4 @@
         </collision>
         <inertial>
-            <!-- <mass value="${wheel_mass}"/>
-            <inertia ixx="0.00000826" ixy="0" ixz="0"
-                     iyy="00.00000826" iyz="0"
-                     izz="0.00000826"/> -->
             <mass value="${physics_config['caster_mass']}"/>
             <inertia ixx="${physics_config['caster_p_ixx']}" ixy="0" ixz="0"
@@ -110,71 +99,34 @@
         <!-- <axis xyz="1 0 0" /> -->
         <limit effort="1000.0" velocity="100.0" />
-        <!-- <dynamics damping="0.01" friction="0.01"/> -->
-        <dynamics damping="${physics_config['wheel_damping']}"
-                        friction="${physics_config['wheel_friction']}"/>
+        <dynamics damping="${physics_config['caster_damping']}"
+                        friction="${physics_config['caster_friction']}"/>
     </joint>
     <!-- Gazebo materials -->
     <gazebo reference="${prefix}_yaw_link">
         <material>Gazebo/Grey</material>
-        <surface>
-            <friction>
-                <ode>
-                    <mu>0.01</mu>
-                    <mu2>0.01</mu2>
-                    <slip1>0.9</slip1>
-                    <slip2>0.9</slip2>
-                </ode>
-            </friction>
-            <contact>
-                <ode>
-                    <kp>100.0</kp>
-                    <kd>1.0</kd>
-                    <soft_cfm>0.01</soft_cfm>
-                    <soft_erp>0.2</soft_erp>
-                </ode>
-            </contact>
-        </surface>
+        <mu>${physics_config['caster_mu']}</mu>
+        <mu2>${physics_config['caster_mu']}</mu2>
+        <slip1>${physics_config['caster_slip']}</slip1>
+        <slip2>${physics_config['caster_slip']}</slip2>
+        <kp>${physics_config['caster_kp']}</kp>
+        <kd>${physics_config['caster_kd']}</kd>
     </gazebo>
     <gazebo reference="${prefix}_roll_link">
         <material>Gazebo/Grey</material>
-        <surface>
-            <friction>
-                <ode>
-                    <mu>0.01</mu>
-                    <mu2>0.01</mu2>
-                    <slip1>0.5</slip1>
-                    <slip2>0.5</slip2>
-                </ode>
-            </friction>
-            <contact>
-                <ode>
-                    <kp>100.0</kp>
-                    <kd>1.0</kd>
-                    <soft_cfm>0.01</soft_cfm>
-                    <soft_erp>0.2</soft_erp>
-                </ode>
-            </contact>
-        </surface>
+        <mu>${physics_config['caster_mu']}</mu>
+        <mu2>${physics_config['caster_mu']}</mu2>
+        <slip1>${physics_config['caster_slip']}</slip1>
+        <slip2>${physics_config['caster_slip']}</slip2>
+        <kp>${physics_config['caster_kp']}</kp>
+        <kd>${physics_config['caster_kd']}</kd>
     </gazebo>
     <gazebo reference="${prefix}_pitch_link">
         <material>Gazebo/Grey</material>
-        <surface>
-            <friction>
-                <ode>
-                    <mu>0.01</mu>
-                    <mu2>0.01</mu2>
-                    <slip1>0.5</slip1>
-                    <slip2>0.5</slip2>
-                </ode>
-            </friction>
-            <contact>
-                <ode>
-                    <kp>100.0</kp>
-                    <kd>1.0</kd>
-                    <soft_cfm>0.01</soft_cfm>
-                    <soft_erp>0.2</soft_erp>
-                </ode>
-            </contact>
-        </surface>
+        <mu>${physics_config['caster_mu']}</mu>
+        <mu2>${physics_config['caster_mu']}</mu2>
+        <slip1>${physics_config['caster_slip']}</slip1>
+        <slip2>${physics_config['caster_slip']}</slip2>
+        <kp>${physics_config['caster_kp']}</kp>
+        <kd>${physics_config['caster_kd']}</kd>
     </gazebo>
   </xacro:macro>

File: xacro/drive_wheel.xacro (robot description, xacro)
@@ -34,24 +34,8 @@
     <gazebo reference="${prefix}_wheel">
         <material>Gazebo/Black</material>
-        <surface>
-            <friction>
-                <ode>
-                    <mu>1.5</mu>
-                    <mu2>1.5</mu2>
-                    <slip1>0.01</slip1>
-                    <slip2>0.01</slip2>
-                </ode>
-            </friction>
-            <contact>
-                <ode>
-                    <kp>1000.0</kp>
-                    <kd>1.0</kd>
-                    <soft_cfm>0.0</soft_cfm>
-                    <soft_erp>0.2</soft_erp>
-                    <max_vel>0.01</max_vel>
-                    <min_depth>0.001</min_depth>
-                </ode>
-            </contact>
-        </surface>
+        <mu>${physics_config['drive_mu']}</mu>
+        <mu2>${physics_config['drive_mu']}</mu2>
+        <kp>${physics_config['drive_kp']}</kp>
+        <kd>${physics_config['drive_kd']}</kd>
     </gazebo>
     <joint name="joint_${prefix}_wheel" type="continuous">

Commit message: bot is little unstable and has linear motion but no angular motion

File: xacro/barista_robot_model.urdf.xacro (robot description, xacro)
@@ -128,6 +128,6 @@
             <max_wheel_torque>${physics_config['max_wheel_torque']}</max_wheel_torque>
             <max_wheel_acceleration>${physics_config['max_wheel_acceleration']}</max_wheel_acceleration>
-            <max_linear_velocity>${physics_config['max_linear_velocity']}</max_linear_velocity>
-            <max_angular_velocity>${physics_config['max_angular_velocity']}</max_angular_velocity>
+            <!-- <max_linear_velocity>${physics_config['max_linear_velocity']}</max_linear_velocity>
+            <max_angular_velocity>${physics_config['max_angular_velocity']}</max_angular_velocity> -->
             <!-- output -->
             <publish_odom>true</publish_odom>

File: xacro/caster_wheel.xacro (robot description, xacro)
@@ -9,6 +9,6 @@
     <xacro:property name="cylinder_length" value="0.010"/>
     <xacro:property name="wheel_mass" value="0.02"/>
-    <!-- <xacro:property name="joint_type" value="fixed"/> -->
-    <xacro:property name="joint_type" value="continuous"/>
+    <xacro:property name="joint_type" value="fixed"/>
+    <!-- <xacro:property name="joint_type" value="continuous"/> -->
     <!-- Yaw link -->
     <link name="${prefix}_yaw_link">

File: xacro/laser_scanner.xacro (robot description, xacro)
@@ -45,5 +45,5 @@
             <sensor type="ray" name="${robot_name}_laser_scanner">
                 <pose>0 0 0 0 0 0</pose>
-                <update_rate>10</update_rate>
+                <update_rate>5</update_rate>
                 <always_on>true</always_on>
                 <visualize>true</visualize>
@@ -51,5 +51,5 @@
                     <scan>
                         <horizontal>
-                            <samples>200</samples>
+                            <samples>100</samples>
                             <resolution>1</resolution>
                             <min_angle>-3.14159</min_angle>
@@ -79,4 +79,5 @@
                     </ros>
                     <frame_name>${robot_name}/laser_optical_frame</frame_name>
+                    <always_on>true</always_on>
                 </plugin>
             </sensor>

Commit message: able to make either linear or angular motion. but not both together. records are being maintained in the value_history.md file

File: xacro/barista_robot_model.urdf.xacro (robot description, xacro)
@@ -58,8 +58,12 @@
         </collision>
         <inertial>
-            <mass value="0.5"/>
-            <inertia ixx="0.002" ixy="0" ixz="0"
-                    iyy="0.002" iyz="0"
-                    izz="0.003"/>
+            <mass value="${physics_config['chassis_mass']}"/>
+            <!-- <inertia ixx="0.0019846" ixy="0" ixz="0"
+                     iyy="0.0019846" iyz="0"
+                     izz="0.0031684"/> -->
+            <inertia ixx="${(1/12) * physics_config['chassis_mass'] * (3 * (base_width/2) * (base_width/2) + base_height * base_height)}"
+                     iyy="${(1/12) * physics_config['chassis_mass'] * (3 * (base_width/2) * (base_width/2) + base_height * base_height)}"
+                     izz="${(1/2) * physics_config['chassis_mass'] * (base_width/2) * (base_width/2)}"
+                     ixy="0" ixz="0" iyz="0"/>
         </inertial>
     </link>
@@ -124,10 +128,11 @@
             <!-- kinematics -->
             <wheel_separation>0.28</wheel_separation>
+            <!-- <wheel_separation>0.24</wheel_separation> -->
             <wheel_diameter>0.0704</wheel_diameter>
             <!-- limits -->
             <max_wheel_torque>${physics_config['max_wheel_torque']}</max_wheel_torque>
             <max_wheel_acceleration>${physics_config['max_wheel_acceleration']}</max_wheel_acceleration>
-            <!-- <max_linear_velocity>${physics_config['max_linear_velocity']}</max_linear_velocity>
-            <max_angular_velocity>${physics_config['max_angular_velocity']}</max_angular_velocity> -->
+            <max_linear_velocity>${physics_config['max_linear_velocity']}</max_linear_velocity>
+            <max_angular_velocity>${physics_config['max_angular_velocity']}</max_angular_velocity>
             <!-- output -->
             <publish_odom>true</publish_odom>
@@ -135,4 +140,5 @@
             <!-- try to remove this later -->
             <publish_wheel_tf>false</publish_wheel_tf>
+            <command_timeout>0.2</command_timeout>
             <odometry_frame>${robot_name}/odom</odometry_frame>
             <robot_base_frame>${robot_name}/base_link</robot_base_frame>

File: xacro/caster_wheel.xacro (robot description, xacro)
@@ -8,5 +8,5 @@
     <xacro:property name="wheel_radius" value="0.0352"/>
     <xacro:property name="cylinder_length" value="0.010"/>
-    <xacro:property name="wheel_mass" value="0.02"/>
+    <!-- <xacro:property name="wheel_mass" value="0.02"/> -->
     <xacro:property name="joint_type" value="fixed"/>
     <!-- <xacro:property name="joint_type" value="continuous"/> -->
@@ -26,7 +26,11 @@
         <inertial>
             <mass value="${physics_config['caster_mass']}"/>
-            <inertia ixx="${physics_config['caster_yr_ixx']}" ixy="0" ixz="0"
+            <!-- <inertia ixx="${physics_config['caster_yr_ixx']}" ixy="0" ixz="0"
                      iyy="${physics_config['caster_yr_iyy']}" iyz="0"
-                     izz="${physics_config['caster_yr_izz']}"/>
+                     izz="${physics_config['caster_yr_izz']}"/> -->
+            <inertia ixx="${(1/12) * physics_config['caster_mass'] * (3 * wheel_radius * wheel_radius + cylinder_length * cylinder_length)}"
+                     iyy="${(1/12) * physics_config['caster_mass'] * (3 * wheel_radius * wheel_radius + cylinder_length * cylinder_length)}"
+                     izz="${(1/2) * physics_config['caster_mass'] * wheel_radius * wheel_radius}"
+                     ixy="0" ixz="0" iyz="0"/>
         </inertial>
     </link>
@@ -56,7 +60,11 @@
         <inertial>
             <mass value="${physics_config['caster_mass']}"/>
-            <inertia ixx="${physics_config['caster_yr_ixx']}" ixy="0" ixz="0"
+            <!-- <inertia ixx="${physics_config['caster_yr_ixx']}" ixy="0" ixz="0"
                      iyy="${physics_config['caster_yr_iyy']}" iyz="0"
-                     izz="${physics_config['caster_yr_izz']}"/>
+                     izz="${physics_config['caster_yr_izz']}"/> -->
+            <inertia ixx="${(1/12) * physics_config['caster_mass'] * (3 * wheel_radius * wheel_radius + cylinder_length * cylinder_length)}"
+                     iyy="${(1/12) * physics_config['caster_mass'] * (3 * wheel_radius * wheel_radius + cylinder_length * cylinder_length)}"
+                     izz="${(1/2) * physics_config['caster_mass'] * wheel_radius * wheel_radius}"
+                     ixy="0" ixz="0" iyz="0"/>
         </inertial>
     </link>
@@ -86,7 +94,11 @@
         <inertial>
             <mass value="${physics_config['caster_mass']}"/>
-            <inertia ixx="${physics_config['caster_p_ixx']}" ixy="0" ixz="0"
+            <!-- <inertia ixx="${physics_config['caster_p_ixx']}" ixy="0" ixz="0"
                      iyy="${physics_config['caster_p_iyy']}" iyz="0"
-                     izz="${physics_config['caster_p_izz']}"/>
+                     izz="${physics_config['caster_p_izz']}"/> -->
+            <inertia ixx="${(2/5) * physics_config['caster_mass'] * wheel_radius * wheel_radius}"
+                     iyy="${(2/5) * physics_config['caster_mass'] * wheel_radius * wheel_radius}"
+                     izz="${(2/5) * physics_config['caster_mass'] * wheel_radius * wheel_radius}"
+                     ixy="0" ixz="0" iyz="0"/>
         </inertial>
     </link>
@@ -97,5 +109,6 @@
         <!-- <axis xyz="0 1 0" /> -->
         <!-- <axis xyz="0 0 1" /> -->
-        <!-- <axis xyz="1 0 0" /> -->
+        <!-- Need to test this -->
+        <!-- <axis xyz="1 0 0" />      -->
         <limit effort="1000.0" velocity="100.0" />
         <dynamics damping="${physics_config['caster_damping']}"

File: xacro/drive_wheel.xacro (robot description, xacro)
@@ -21,13 +21,17 @@
         </collision>
         <inertial>
-            <!-- <mass value="0.05"/>
-            <inertia ixx="0.000005752" ixy="0" ixz="0"
-                    iyy="0.000005752" iyz="0"
-                    izz="0.000010325"/> -->
             <mass value="${physics_config['wheel_mass']}"/>
-            <inertia ixx="${physics_config['wheel_mass'] * physics_config['wheel_ixx_factor']}"
+            <!-- <inertia ixx="${physics_config['wheel_ixx_factor']}"
+                     iyy="${physics_config['wheel_iyy_factor']}"
+                     izz="${physics_config['wheel_izz_factor']}"
+                     ixy="0" ixz="0" iyz="0"/> -->
+            <inertia ixx="${(1/12) * physics_config['wheel_mass'] * (3 * wheel_radius * wheel_radius + wheel_width * wheel_width)}"
+                     iyy="${(1/12) * physics_config['wheel_mass'] * (3 * wheel_radius * wheel_radius + wheel_width * wheel_width)}"
+                     izz="${(1/2) * physics_config['wheel_mass'] * wheel_radius * wheel_radius}"
+                     ixy="0" ixz="0" iyz="0"/>
+            <!-- <inertia ixx="${physics_config['wheel_mass'] * physics_config['wheel_ixx_factor']}"
                     iyy="${physics_config['wheel_mass'] * physics_config['wheel_iyy_factor']}"
                     izz="${physics_config['wheel_mass'] * physics_config['wheel_izz_factor']}"
-                    ixy="0" ixz="0" iyz="0"/>
+                    ixy="0" ixz="0" iyz="0"/> -->
         </inertial>
     </link>
@@ -36,4 +40,6 @@
         <mu>${physics_config['drive_mu']}</mu>
         <mu2>${physics_config['drive_mu']}</mu2>
+        <slip1>${physics_config['drive_slip']}</slip1>
+        <slip2>${physics_config['drive_slip']}</slip2>
         <kp>${physics_config['drive_kp']}</kp>
         <kd>${physics_config['drive_kd']}</kd>

File: xacro/laser_scanner.xacro (robot description, xacro)
@@ -33,5 +33,7 @@
         <!-- Laser joint -->
         <joint name="joint_laser" type="fixed">
-            <origin xyz="0.12 0.0 0.077" rpy="0.0 0.0 0.0"/>
+            <!-- <origin xyz="0.12 0.0 0.077" rpy="0.0 0.0 0.0"/> -->
+            <!-- <origin xyz="-0.12 0.0 0.077" rpy="0.0 0.0 0.0"/> -->
+            <origin xyz="-0.12 0.0 0.077" rpy="0.0 0.0 3.14159"/>
             <parent link="chassis"/>
             <child link="laser_link"/>
