Commit message: got working angular and linear motion (with little to no noise). Fixing 'Try7' values.

File: xacro/barista_robot_model.urdf.xacro (robot description, xacro)
@@ -76,4 +76,19 @@
         <material>${colour}</material>
     </gazebo>
+    <!-- FRONT indicator -->
+    <link name="front_indicator">
+        <visual>
+            <origin xyz="0 0 0" rpy="0 0 0"/>
+            <geometry>
+                <box size="0.10 0.01 0.01"/>
+            </geometry>
+            <material name="green_light"/>
+        </visual>
+    </link>
+    <joint name="joint_front_indicator" type="fixed">
+        <origin xyz="-0.09 0.0 0.05" rpy="0.0 0.0 0.0"/>
+        <parent link="cup_holder_tray"/>
+        <child link="front_indicator"/>
+    </joint>
     <!-- Drive Wheel -->
     <xacro:include filename="$(find barista_robot_description)/xacro/drive_wheel.xacro"/>
@@ -128,11 +143,10 @@
             <!-- kinematics -->
             <wheel_separation>0.28</wheel_separation>
-            <!-- <wheel_separation>0.24</wheel_separation> -->
             <wheel_diameter>0.0704</wheel_diameter>
             <!-- limits -->
             <max_wheel_torque>${physics_config['max_wheel_torque']}</max_wheel_torque>
-            <max_wheel_acceleration>${physics_config['max_wheel_acceleration']}</max_wheel_acceleration>
+            <!-- <max_wheel_acceleration>${physics_config['max_wheel_acceleration']}</max_wheel_acceleration> -->
             <max_linear_velocity>${physics_config['max_linear_velocity']}</max_linear_velocity>
-            <max_angular_velocity>${physics_config['max_angular_velocity']}</max_angular_velocity>
+            <!-- <max_angular_velocity>${physics_config['max_angular_velocity']}</max_angular_velocity> -->
             <!-- output -->
             <publish_odom>true</publish_odom>

File: xacro/caster_wheel.xacro (robot description, xacro)
@@ -41,5 +41,5 @@
         <!-- <axis xyz="0 1 0" /> -->
         <axis xyz="0 0 1 " />
-        <limit effort="1000.0" velocity="100.0" />
+        <!-- <limit effort="1000.0" velocity="100.0" /> -->
         <dynamics damping="${physics_config['caster_damping']}"
                         friction="${physics_config['caster_friction']}"/>
@@ -75,5 +75,5 @@
         <!-- <axis xyz="1 0 0" /> -->
         <axis xyz="0 1 0" />
-        <limit effort="1000.0" velocity="100.0" />
+        <!-- <limit effort="1000.0" velocity="100.0" /> -->
         <dynamics damping="${physics_config['caster_damping']}"
                         friction="${physics_config['caster_friction']}"/>
@@ -111,5 +111,5 @@
         <!-- Need to test this -->
         <!-- <axis xyz="1 0 0" />      -->
-        <limit effort="1000.0" velocity="100.0" />
+        <!-- <limit effort="1000.0" velocity="100.0" /> -->
         <dynamics damping="${physics_config['caster_damping']}"
                         friction="${physics_config['caster_friction']}"/>

File: xacro/drive_wheel.xacro (robot description, xacro)
@@ -50,6 +50,6 @@
         <parent link="chassis"/>
         <axis rpy="0 0 0" xyz="0 0 1"/>
-        <limit effort="10000" velocity="1000"/>
-        <!-- <joint_properties damping="3.0" friction="0.4"/> -->
+        <!-- this effor was the main issue. use it only for primatic and revolute joint -->
+        <!-- <limit effort="10000" velocity="1000"/> -->
         <joint_properties damping="${physics_config['wheel_damping']}"
                         friction="${physics_config['wheel_friction']}"/>

File: xacro/laser_scanner.xacro (robot description, xacro)
@@ -47,5 +47,5 @@
             <sensor type="ray" name="${robot_name}_laser_scanner">
                 <pose>0 0 0 0 0 0</pose>
-                <update_rate>5</update_rate>
+                <update_rate>10</update_rate>
                 <always_on>true</always_on>
                 <visualize>true</visualize>

Commit message: CP8 Task1 tested and verified. code cleanup done

File: xacro/barista_robot_model.urdf.xacro (robot description, xacro)
@@ -59,7 +59,4 @@
         <inertial>
             <mass value="${physics_config['chassis_mass']}"/>
-            <!-- <inertia ixx="0.0019846" ixy="0" ixz="0"
-                     iyy="0.0019846" iyz="0"
-                     izz="0.0031684"/> -->
             <inertia ixx="${(1/12) * physics_config['chassis_mass'] * (3 * (base_width/2) * (base_width/2) + base_height * base_height)}"
                      iyy="${(1/12) * physics_config['chassis_mass'] * (3 * (base_width/2) * (base_width/2) + base_height * base_height)}"
@@ -83,5 +80,5 @@
                 <box size="0.10 0.01 0.01"/>
             </geometry>
-            <material name="green_light"/>
+            <material name="white"/>
         </visual>
     </link>
@@ -146,7 +143,5 @@
             <!-- limits -->
             <max_wheel_torque>${physics_config['max_wheel_torque']}</max_wheel_torque>
-            <!-- <max_wheel_acceleration>${physics_config['max_wheel_acceleration']}</max_wheel_acceleration> -->
             <max_linear_velocity>${physics_config['max_linear_velocity']}</max_linear_velocity>
-            <!-- <max_angular_velocity>${physics_config['max_angular_velocity']}</max_angular_velocity> -->
             <!-- output -->
             <publish_odom>true</publish_odom>

File: xacro/caster_wheel.xacro (robot description, xacro)
@@ -8,5 +8,4 @@
     <xacro:property name="wheel_radius" value="0.0352"/>
     <xacro:property name="cylinder_length" value="0.010"/>
-    <!-- <xacro:property name="wheel_mass" value="0.02"/> -->
     <xacro:property name="joint_type" value="fixed"/>
     <!-- <xacro:property name="joint_type" value="continuous"/> -->
@@ -26,7 +25,4 @@
         <inertial>
             <mass value="${physics_config['caster_mass']}"/>
-            <!-- <inertia ixx="${physics_config['caster_yr_ixx']}" ixy="0" ixz="0"
-                     iyy="${physics_config['caster_yr_iyy']}" iyz="0"
-                     izz="${physics_config['caster_yr_izz']}"/> -->
             <inertia ixx="${(1/12) * physics_config['caster_mass'] * (3 * wheel_radius * wheel_radius + cylinder_length * cylinder_length)}"
                      iyy="${(1/12) * physics_config['caster_mass'] * (3 * wheel_radius * wheel_radius + cylinder_length * cylinder_length)}"
@@ -39,7 +35,5 @@
         <parent link="chassis" />
         <child link="${prefix}_yaw_link" />
-        <!-- <axis xyz="0 1 0" /> -->
         <axis xyz="0 0 1 " />
-        <!-- <limit effort="1000.0" velocity="100.0" /> -->
         <dynamics damping="${physics_config['caster_damping']}"
                         friction="${physics_config['caster_friction']}"/>
@@ -60,7 +54,4 @@
         <inertial>
             <mass value="${physics_config['caster_mass']}"/>
-            <!-- <inertia ixx="${physics_config['caster_yr_ixx']}" ixy="0" ixz="0"
-                     iyy="${physics_config['caster_yr_iyy']}" iyz="0"
-                     izz="${physics_config['caster_yr_izz']}"/> -->
             <inertia ixx="${(1/12) * physics_config['caster_mass'] * (3 * wheel_radius * wheel_radius + cylinder_length * cylinder_length)}"
                      iyy="${(1/12) * physics_config['caster_mass'] * (3 * wheel_radius * wheel_radius + cylinder_length * cylinder_length)}"
@@ -73,7 +64,5 @@
         <parent link="${prefix}_yaw_link" />
         <child link="${prefix}_roll_link" />
-        <!-- <axis xyz="1 0 0" /> -->
         <axis xyz="0 1 0" />
-        <!-- <limit effort="1000.0" velocity="100.0" /> -->
         <dynamics damping="${physics_config['caster_damping']}"
                         friction="${physics_config['caster_friction']}"/>
@@ -94,7 +83,4 @@
         <inertial>
             <mass value="${physics_config['caster_mass']}"/>
-            <!-- <inertia ixx="${physics_config['caster_p_ixx']}" ixy="0" ixz="0"
-                     iyy="${physics_config['caster_p_iyy']}" iyz="0"
-                     izz="${physics_config['caster_p_izz']}"/> -->
             <inertia ixx="${(2/5) * physics_config['caster_mass'] * wheel_radius * wheel_radius}"
                      iyy="${(2/5) * physics_config['caster_mass'] * wheel_radius * wheel_radius}"
@@ -107,9 +93,4 @@
         <parent link="${prefix}_roll_link" />
         <child link="${prefix}_pitch_link" />
-        <!-- <axis xyz="0 1 0" /> -->
-        <!-- <axis xyz="0 0 1" /> -->
-        <!-- Need to test this -->
-        <!-- <axis xyz="1 0 0" />      -->
-        <!-- <limit effort="1000.0" velocity="100.0" /> -->
         <dynamics damping="${physics_config['caster_damping']}"
                         friction="${physics_config['caster_friction']}"/>

File: xacro/drive_wheel.xacro (robot description, xacro)
@@ -22,16 +22,8 @@
         <inertial>
             <mass value="${physics_config['wheel_mass']}"/>
-            <!-- <inertia ixx="${physics_config['wheel_ixx_factor']}"
-                     iyy="${physics_config['wheel_iyy_factor']}"
-                     izz="${physics_config['wheel_izz_factor']}"
-                     ixy="0" ixz="0" iyz="0"/> -->
             <inertia ixx="${(1/12) * physics_config['wheel_mass'] * (3 * wheel_radius * wheel_radius + wheel_width * wheel_width)}"
                      iyy="${(1/12) * physics_config['wheel_mass'] * (3 * wheel_radius * wheel_radius + wheel_width * wheel_width)}"
                      izz="${(1/2) * physics_config['wheel_mass'] * wheel_radius * wheel_radius}"
                      ixy="0" ixz="0" iyz="0"/>
-            <!-- <inertia ixx="${physics_config['wheel_mass'] * physics_config['wheel_ixx_factor']}"
-                    iyy="${physics_config['wheel_mass'] * physics_config['wheel_iyy_factor']}"
-                    izz="${physics_config['wheel_mass'] * physics_config['wheel_izz_factor']}"
-                    ixy="0" ixz="0" iyz="0"/> -->
         </inertial>
     </link>
@@ -50,6 +42,4 @@
         <parent link="chassis"/>
         <axis rpy="0 0 0" xyz="0 0 1"/>
-        <!-- this effor was the main issue. use it only for primatic and revolute joint -->
-        <!-- <limit effort="10000" velocity="1000"/> -->
         <joint_properties damping="${physics_config['wheel_damping']}"
                         friction="${physics_config['wheel_friction']}"/>

File: xacro/laser_scanner.xacro (robot description, xacro)
@@ -18,6 +18,4 @@
             </collision>
             <inertial>
-                <!-- <mass value="0.3"/>
-                <inertia ixx="0.001" ixy="0" ixz="0" iyy="0.001" iyz="0" izz="0.0005"/> -->
                 <mass value="0.01"/>
                 <inertia ixx="6.066578520833334e-06" ixy="0" ixz="0" iyy="6.072950163333333e-06" iyz="0" izz="9.365128684166666e-06"/>
@@ -33,6 +31,4 @@
         <!-- Laser joint -->
         <joint name="joint_laser" type="fixed">
-            <!-- <origin xyz="0.12 0.0 0.077" rpy="0.0 0.0 0.0"/> -->
-            <!-- <origin xyz="-0.12 0.0 0.077" rpy="0.0 0.0 0.0"/> -->
             <origin xyz="-0.12 0.0 0.077" rpy="0.0 0.0 3.14159"/>
             <parent link="chassis"/>
