Commit message: Increased laser rays and changed spawning position

File: xacro/laser_scanner.xacro (robot description, xacro)
@@ -49,6 +49,7 @@
                     <scan>
                         <horizontal>
-                            <samples>100</samples>
+                            <samples>260</samples>
                             <resolution>1</resolution>
+                            <!-- <resolution>2</resolution> -->
                             <min_angle>-3.14159</min_angle>
                             <max_angle>3.14159</max_angle>

File: xacro/physics_properties.xacro (robot description, xacro)
@@ -3,4 +3,5 @@
     <!-- Load once, use everywhere -->
     <xacro:property name="config_file" value="$(find barista_robot_description)/config/robot_physics.yaml"/>
-    <xacro:property name="physics_config" value="${load_yaml(config_file)['robot_physics']}"/>
+    <!-- <xacro:property name="physics_config" value="${load_yaml(config_file)['robot_physics']}"/> -->
+    <xacro:property name="physics_config" value="${xacro.load_yaml(config_file)['robot_physics']}"/>
 </robot>
