Commit message: loading yaml through xacro.loadyaml not working on cloud. so changing it back to load_yaml

File: xacro/physics_properties.xacro (robot description, xacro)
@@ -3,5 +3,5 @@
     <!-- Load once, use everywhere -->
     <xacro:property name="config_file" value="$(find barista_robot_description)/config/robot_physics.yaml"/>
-    <!-- <xacro:property name="physics_config" value="${load_yaml(config_file)['robot_physics']}"/> -->
-    <xacro:property name="physics_config" value="${xacro.load_yaml(config_file)['robot_physics']}"/>
+    <xacro:property name="physics_config" value="${load_yaml(config_file)['robot_physics']}"/>
+    <!-- <xacro:property name="physics_config" value="${xacro.load_yaml(config_file)['robot_physics']}"/> -->
 </robot>
